File: Embedded-Light/Hardware/f7-ginger/ginger.sch (KiCad schematic (older format))
At the start: 108 parts, among them P1 CONN_02X20, P2 3V_IN, P3 USB_OTG, P4 USB_OTG, P5 USB_OTG, P6 AuxPwrSel, SW1 Reset, SW10 B, SW11 B, SW12 B, SW13 B, SW14 B, SW15 B, SW16 B, SW17 B, SW18 B, SW19 B, SW2 B, SW20 B, SW21 B, SW3 B, SW4 B, SW5 B, SW6 B, SW7 B, SW8 B, SW9 B, U1 STM32F746BGTx, U2 MICROSD, U3 FT232RL, U4 FT232RL, U5 LM2937-3.3, Y1 20MHz

Commit message: Ginger: updated schematics to the current real board state.
Parts:
- added P?: SWD, symbol CONN_01X04
- added R?: 10k, Resistors_SMD:R_0805, symbol R
- R1: value 330 -> 22
Connections:
- net +3V3: now also R?.1
- net GND: now also P?.2 (P2)
- net tft_rd: no longer P1.11 (P11)
- net at U1.147 (PA13): now also P?.3 (P3)
- net at U1.159 (PA14): now also P?.1 (P1)
- net cpu_reset: now reaches R3.2, SW1.2, U1.34 (NRST)
- net cpu_reset: now also P?.4 (P4)
- new net: P1.11 (P11), R?.2
- no-connect marks 132 -> 130
Changed lines of the file:
@@
 $EndComp
 NoConn ~ 9700 2350
-NoConn ~ 9500 2350
 NoConn ~ 9400 2350
 NoConn ~ 9300 2350
@@
 NoConn ~ 10200 3250
 NoConn ~ 10200 3350
-NoConn ~ 10200 3750
 NoConn ~ 8700 2350
 NoConn ~ 6400 2350
@@
 P 1150 4650
 F 0 "R1" V 1230 4650 50  0000 C CNN
-F 1 "330" V 1150 4650 50  0000 C CNN
+F 1 "22" V 1150 4650 50  0000 C CNN
 F 2 "Resistors_SMD:R_0805" V 1080 4650 50  0001 C CNN
 F 3 "" H 1150 4650 50  0000 C CNN
@@
 	1    0    0    -1
 $EndComp
-Text Label 1500 3350 2    60   ~ 0
-tft_rd
+$Comp
+L R R?
+U 1 1 5B421015
+P 1050 3350
+F 0 "R?" V 1130 3350 50  0000 C CNN
+F 1 "10k" V 1050 3350 50  0000 C CNN
+F 2 "Resistors_SMD:R_0805" V 980 3350 50  0001 C CNN
+F 3 "" H 1050 3350 50  0000 C CNN
+	1    1050 3350
+	0    -1   1    0
+$EndComp
+Wire Wire Line
+	900  3350 800  3350
+Connection ~ 800  3350
+Wire Wire Line
+	1200 3350 1500 3350
+$Comp
+L CONN_01X04 P?
+U 1 1 5B424BEC
+P 11650 1350
+F 0 "P?" H 11650 1600 50  0000 C CNN
+F 1 "SWD" V 11750 1350 50  0000 C CNN
+F 2 "" H 11650 1350 50  0000 C CNN
+F 3 "" H 11650 1350 50  0000 C CNN
+	1    11650 1350
+	1    0    0    -1
+$EndComp
+Wire Wire Line
+	9500 2350 9500 1750
+Wire Wire Line
+	9500 1750 10450 1750
+Wire Wire Line
+	10450 1750 10450 1200
+Wire Wire Line
+	10450 1200 11450 1200
+$Comp
+L GND #PWR?
+U 1 1 5B428A4D
+P 10850 1600
+F 0 "#PWR?" H 10850 1350 50  0001 C CNN
+F 1 "GND" H 10850 1450 50  0000 C CNN
+F 2 "" H 10850 1600 50  0000 C CNN
+F 3 "" H 10850 1600 50  0000 C CNN
+	1    10850 1600
+	1    0    0    -1
+$EndComp
+Wire Wire Line
+	10850 1300 11450 1300
+Wire Wire Line
+	10200 3750 10600 3750
+Wire Wire Line
+	10600 3750 10600 1400
+Wire Wire Line
+	10600 1400 11450 1400
+Text Label 3800 5800 2    60   ~ 0
+cpu_reset
+Text Label 11450 1500 2    60   ~ 0
+cpu_reset
+Wire Wire Line
+	10850 1300 10850 1600
 $EndSCHEMATC

Commit message: Ginger: schematic sheet updated with TODOs.
Parts:
- R20: value 330 -> 510
Other:
- note added: "TODO: 4-bit bus"
- note added: "TODO: SWD connector"
- note added: "TODO: connect TFT_RD to 3V3 via 10k res.\nand optional DNP placeholder to connect to MCU's FMC_OE."
- note added: "TODO: in case of using the battery power, it's pretty safe to remove a half of these capacitors."
- note added: "TODO: more user LEDs (at least 2 more)."
- note added: "TODO: remove "weak" power input."
- note added: "TODO: remove R5. Connect each cathode via\ndarlington pair (ULN2003A) + 330Ohm res."
- note added: "TODO: remove UART3 channel"
- note added: "TODO: replace jumper with button"
- note added: "TODO: replace mini USB with micro USB, or even better: USB A."
Changed lines of the file:
@@
 P 5500 11850
 F 0 "R20" V 5580 11850 50  0000 C CNN
-F 1 "330" V 5500 11850 50  0000 C CNN
+F 1 "510" V 5500 11850 50  0000 C CNN
 F 2 "Resistors_SMD:R_0805" V 5430 11850 50  0001 C CNN
 F 3 "" H 5500 11850 50  0000 C CNN
@@
 Wire Wire Line
 	10850 1300 10850 1600
+Text Notes 3900 950  0    60   ~ 0
+TODO: replace jumper with button
+Text Notes 650  5050 0    60   ~ 0
+TODO: connect TFT_RD to 3V3 via 10k res.\nand optional DNP placeholder to connect to MCU's FMC_OE.
+Text Notes 2100 10650 0    60   ~ 0
+TODO: remove R5. Connect each cathode via\ndarlington pair (ULN2003A) + 330Ohm res.
+Text Notes 8600 10400 0    60   ~ 0
+TODO: remove UART3 channel
+Text Notes 11900 1300 0    60   ~ 0
+TODO: SWD connector
+Text Notes 9600 11250 0    60   ~ 0
+TODO: remove "weak" power input.
+Text Notes 4500 13750 0    60   ~ 0
+TODO: in case of using the battery power, it's pretty safe to remove a half of these capacitors.
+Text Notes 10100 8200 0    60   ~ 0
+TODO: more user LEDs (at least 2 more).
+Text Notes 10350 750  0    60   ~ 0
+TODO: 4-bit bus
+Text Notes 12550 5150 0    60   ~ 0
+TODO: replace mini USB with micro USB, or even better: USB A.
 $EndSCHEMATC

Commit message: Ginger: keyboard tested.
Other:
- note added: "TODO: segments 12 and 13 should be swapped!"
Changed lines of the file:
@@
 Text Notes 12550 5150 0    60   ~ 0
 TODO: replace mini USB with micro USB, or even better: USB A.
+Text Notes 2100 10900 0    60   ~ 0
+TODO: segments 12 and 13 should be swapped!
 $EndSCHEMATC

Commit message: Ginger board: added note about RXTX LEDs.
Parts:
- D2: value TX -> RX
- D4: value RX -> TX
Other:
- note added: "RX & TX leds should be inverted, since they're showing PC side"
Changed lines of the file:
@@
 P 11850 3150
 F 0 "D4" H 11600 3050 50  0000 C CNN
-F 1 "RX" H 11850 3050 50  0000 C CNN
+F 1 "TX" H 11850 3050 50  0000 C CNN
 F 2 "Resistors_SMD:R_1210" H 11850 3150 50  0001 C CNN
 F 3 "" H 11850 3150 50  0000 C CNN
@@
 P 11350 3250
 F 0 "D2" H 11350 3350 50  0000 C CNN
-F 1 "TX" H 11350 3150 50  0000 C CNN
+F 1 "RX" H 11350 3150 50  0000 C CNN
 F 2 "Resistors_SMD:R_1210" H 11350 3250 50  0001 C CNN
 F 3 "" H 11350 3250 50  0000 C CNN
@@
 Text Notes 2100 10900 0    60   ~ 0
 TODO: segments 12 and 13 should be swapped!
+Text Notes 10950 2100 0    60   ~ 0
+RX & TX leds should be inverted, since they're showing PC side
 $EndSCHEMATC
