File: Embedded-Light/Hardware/f7-ginger2/ginger2.sch (KiCad schematic (older format))
At the start: 74 parts, among them P1 USB_OTG, P2 USB_A, P3 SWD, P4 microSD, P5 BATR, SW1 RST, SW2 B4, SW3 B3, SW4 B2, SW5 B1, SW6 BOOT, U3 ULN2003A, U5 STM32F767IIT6, U6 FT232RL, U7 LM2937-3.3, U8 WF24HTLAJDNN0, U9 DT022CTFT, Y1 20MHz

Commit message: Ginger2: new board schematics and placement, ready to route.
Parts:
- removed C21, C22: 47u, Capacitors_Tantalum_SMD:TantalC_SizeB_EIA-3528_Wave, symbol CP1
- removed D4: RX, Resistors_SMD:R_1210, symbol LED
- removed D5: TX, Resistors_SMD:R_1210, symbol LED
- removed D6: 3V, Resistors_SMD:R_1210, symbol LED
- removed P1: USB_OTG, Connect:USB_Mini-B, symbol USB_OTG
- removed R30, R53: 1k, Resistors_SMD:R_0805, symbol R
- removed R33, R35: 510, Resistors_SMD:R_0805, symbol R
- removed R38, R39, R48: 330, Resistors_SMD:R_0805, symbol R
- removed R40, R43, R44, R46: 0, Resistors_SMD:R_0402, symbol R
- removed R41, R42, R45, R47: DNP, Resistors_SMD:R_0402, symbol R
- removed SW6: BOOT, button_bourns:but_7914G, symbol SW_PUSH_SMALL
- removed U3: ULN2003A, Housings_SOIC:SOIC-16_3.9x9.9mm_Pitch1.27mm, symbol ULN2003A
- removed U6: FT232RL, Housings_SSOP:SSOP-28_5.3x10.2mm_Pitch0.65mm, symbol FT232RL
- removed U7: LM2937-3.3, TO_SOT_Packages_THT:TO-220_Neutral123_Horizontal, symbol LM7805CT
- removed U9: DT022CTFT, XF2M45151A:XF2M45151A, symbol DT022CTFT
- removed W1: MCO, Connect:PINTST, symbol TEST_1P
- added C21: 4.7u, Capacitors_SMD:C_0805, symbol C
- added C22: 10n, Capacitors_SMD:C_0805, symbol C
- added C23: 100n, Capacitors_SMD:C_0805, symbol C
- added C24: 10u, Capacitors_SMD:C_0805, symbol C
- added L1: 2.2uH, Resistors_SMD:R_0805, symbol L_Small
- added P1: UART, Pin_Headers:Pin_Header_Straight_1x04, symbol CONN_01X04
- added Q1: FDN337N, TO_SOT_Packages_SMD:SOT-23, symbol Q_NMOS_GSD
- added R2, R4: 10k, Resistors_SMD:R_0805, symbol R
- added R5: 1k, Resistors_SMD:R_0805, symbol R
- added R6: 510, Resistors_SMD:R_0805, symbol R
- added U4: LM3671MF-FIX, TO_SOT_Packages_SMD:SOT-23-5, symbol LM3671MF-FIX
- added U5: LP2985LV, TO_SOT_Packages_SMD:SOT-23-5, symbol LP2985LV
- D3: value 5V -> PWR
- P2: value USB_A -> USB_HOST
- P5: value BATR -> BAT
- R1: value 0 -> 1k; footprint Resistors_SMD:R_0402 -> Resistors_SMD:R_0805
- renumbered DD7 to U1, U5 to U2, U8 to U3
Connections:
- net LCD1_LK3 is gone; now on net LCD1_LK1: U3.36 (LEDK3), U3.37 (LEDK4)
- net +3V3: now also D3.2 (A), C24.1, L1.2, U4.4 (FB)
- net +5V: now also C23.1, U5.5 (VOUT); no longer D3.2 (A), P5.1 (P1), R1.2
- net GND: now also C21.2, C22.2, C23.2, C24.2, P1.4 (P4), Q1.2 (S), R2.2, R4.2, R6.1, U4.2 (GND), U5.2 (GND); no longer U1.28 (VSS)
- net LCD1_LK1: now also Q1.3 (D)
- net cpu_boot: now also R1.1
- net usb_pon: now reaches U2.54 (PC4)
- net usb_pon: now also R4.1, U5.3 (ON/OFF)
- net at D3.1 (K): now also R6.2
- net lcd_b2: no longer names the net of U2.150 (PD6/LTDC_B2)
- net lcd_b3: no longer names the net of U2.154 (PG11/LTDC_B3)
- net lcd_b4: no longer names the net of U2.155 (PG12/LTDC_B4)
- net lcd_b5: no longer names the net of U2.47 (PA3/LTDC_B5)
- net lcd_b6: no longer names the net of U2.167 (PB8/LTDC_B6)
- net lcd_b7: no longer names the net of U2.168 (PB9/LTDC_B7)
- net lcd_clk: no longer names the net of U2.111 (PG7/LTDC_CLK)
- net lcd_enable: no longer names the net of U2.28 (PF10/LTDC_DE)
- net lcd_g2: no longer names the net of U2.128 (PH13/LTDC_G2)
- net lcd_g3: no longer names the net of U2.129 (PH14/LTDC_G3)
- net lcd_g4: no longer names the net of U2.45 (PH4/LTDC_G4)
- net lcd_g5: no longer names the net of U2.80 (PB11/LTDC_G5)
- net lcd_g6: no longer names the net of U2.13 (PI11/LTDC_G6)
- net lcd_g7: no longer names the net of U2.133 (PI2/LTDC_G7)
- net lcd_hs: no longer names the net of U2.12 (PI10/LTDC_HSYNC)
- net lcd_r2: no longer names the net of U2.41 (PA1/LTDC_R2)
- net lcd_r3: no longer names the net of U2.56 (PB0/LTDC_R3)
- net lcd_r4: no longer names the net of U2.87 (PH10/LTDC_R4)
- net lcd_r5: no longer names the net of U2.88 (PH11/LTDC_R5)
- net lcd_r6: no longer names the net of U2.57 (PB1/LTDC_R6)
- net lcd_r7: no longer names the net of U2.110 (PG6/LTDC_R7)
- net lcd_rst: no longer names the net of U2.84 (PH7/LCD2_RESET)
- net lcd_vs: no longer names the net of U2.11 (PI9/LTDC_VSYNC)
- net pwm_ch1: no longer names the net of U2.40 (PA0/WKUP/TIM2_CH1)
- net pwm_ch1: now also Q1.1 (G), R2.1
- net uart_rx: no longer names the net of U2.121 (PA10/USART1_RX)
- net uart_rx: now also P1.1 (P1)
- net uart_tx: no longer names the net of U2.120 (PA9/USART1_TX)
- net uart_tx: now also P1.2 (P2)
- new net: P1.3 (P3), R1.2
- new net: C21.1, P5.1 (P1), R5.1, U4.1 (Vin), U5.1 (VIN)
- new net: C22.1, U5.4 (BYPASS)
- new net: R5.2, U4.3 (En)
- new net: L1.1, U4.5 (SW)
- no-connect marks 68 -> 73
Other:
- moved on the sheet: C1, C10, C11, C12, C13, C14, C15, C16, C17, C18, C19, C2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

Commit message: Ginger-2: updated schematics for future board revision
Parts:
- removed P2: USB_HOST, Connect:USB_A, symbol USB_A
- added R?: 0, Resistors_SMD:R_0402, symbol R
- added R? (x16): 10k, Resistors_SMD:R_0805, symbol R
- added SW? (x64): B, symbol SW_PUSH_SMALL
Connections:
- net GND: now also R?.1, R?.1, R?.1, R?.1, R?.1, R?.1, R?.1, R?.1, R?.2, R?.2, R?.2, R?.2, R?.2, R?.2, R?.2, R?.2, R?.2; no longer Q1.2 (S)
- new net: Q1.2 (S), R?.1
- new net kbd_c1: R?.2, SW?.2, SW?.2, SW?.2, SW?.2, SW?.2, SW?.2, SW?.2, SW?.2
- new net kbd_c2: R?.2, SW?.2, SW?.2, SW?.2, SW?.2, SW?.2, SW?.2, SW?.2, SW?.2
- new net kbd_c3: R?.2, SW?.2, SW?.2, SW?.2, SW?.2, SW?.2, SW?.2, SW?.2, SW?.2
- new net kbd_c4: R?.2, SW?.2, SW?.2, SW?.2, SW?.2, SW?.2, SW?.2, SW?.2, SW?.2
- new net kbd_c5: R?.2, SW?.2, SW?.2, SW?.2, SW?.2, SW?.2, SW?.2, SW?.2, SW?.2
- new net kbd_c6: R?.2, SW?.2, SW?.2, SW?.2, SW?.2, SW?.2, SW?.2, SW?.2, SW?.2
- new net kbd_c7: R?.2, SW?.2, SW?.2, SW?.2, SW?.2, SW?.2, SW?.2, SW?.2, SW?.2
- new net kbd_c8: R?.2, SW?.2, SW?.2, SW?.2, SW?.2, SW?.2, SW?.2, SW?.2, SW?.2
- new net kbd_l1: R?.1, SW?.1, SW?.1, SW?.1, SW?.1, SW?.1, SW?.1, SW?.1, SW?.1
- new net kbd_l2: R?.1, SW?.1, SW?.1, SW?.1, SW?.1, SW?.1, SW?.1, SW?.1, SW?.1
- new net kbd_l3: R?.1, SW?.1, SW?.1, SW?.1, SW?.1, SW?.1, SW?.1, SW?.1, SW?.1
- new net kbd_l4: R?.1, SW?.1, SW?.1, SW?.1, SW?.1, SW?.1, SW?.1, SW?.1, SW?.1
- new net kbd_l5: R?.1, SW?.1, SW?.1, SW?.1, SW?.1, SW?.1, SW?.1, SW?.1, SW?.1
- new net kbd_l6: R?.1, SW?.1, SW?.1, SW?.1, SW?.1, SW?.1, SW?.1, SW?.1, SW?.1
- new net kbd_l7: R?.1, SW?.1, SW?.1, SW?.1, SW?.1, SW?.1, SW?.1, SW?.1, SW?.1
- new net kbd_l8: R?.1, SW?.1, SW?.1, SW?.1, SW?.1, SW?.1, SW?.1, SW?.1, SW?.1
- no-connect marks 73 -> 75
Other:
- moved on the sheet: C1, C10, C11, C12, C13, C14, C15, C16, C17, C18, C19, C2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
