File: Embedded-Light/Hardware/Helga/bottom.sch (KiCad schematic (older format))
At the start: 80 parts

Commit message: Helga: schematics updated
Parts:
- added D?: PWR, symbol LED
- added R?: 510, symbol R
- added SW?: Power, symbol SWITCH_INV
- added W?: AAA_POS1, symbol TEST_1P
- added W?: AAA_NEG1, symbol TEST_1P
- added W?: AAA_POS2, symbol TEST_1P
- added W?: AAA_NEG2, symbol TEST_1P
- added W?: AAA_POS3, symbol TEST_1P
- added W?: AAA_NEG3, symbol TEST_1P
Connections:
- net GNDA: now also R?.2, W?.1
- net VPP: now also D?.2 (A), SW?.2
- new net: W?.1, W?.1 (x2)
- new net: SW?.1, W?.1
- new net: D?.1 (K), R?.1
- no-connect marks 0 -> 1
Other:
- note added: "Battery pack"
- moved on the sheet: R?, SW?
