File: Embedded-Light/Hardware/Helga/helga.sch (KiCad schematic (older format))
At the start: 2 parts

Commit message: Helga: schematics updated
Connections:
- net Top Side/CPIN1: now reaches P?.1 (P1)
- net Top Side/CPIN10: now reaches P?.10 (P10)
- net Top Side/CPIN11: now reaches P?.11 (P11)
- net Top Side/CPIN12: now reaches P?.12 (P12)
- net Top Side/CPIN13: now reaches P?.13 (P13)
- net Top Side/CPIN14: now reaches P?.14 (P14)
- net Top Side/CPIN15: now reaches P?.15 (P15)
- net Top Side/CPIN16: now reaches P?.16 (P16)
- net Top Side/CPIN17: now reaches P?.17 (P17)
- net Top Side/CPIN18: now reaches P?.18 (P18)
- net Top Side/CPIN19: now reaches P?.19 (P19)
- net Top Side/CPIN2: now reaches P?.2 (P2)
- net Top Side/CPIN20: now reaches P?.20 (P20)
- net Top Side/CPIN3: now reaches P?.3 (P3)
- net Top Side/CPIN4: now reaches P?.4 (P4)
- net Top Side/CPIN5: now reaches P?.5 (P5)
- net Top Side/CPIN6: now reaches P?.6 (P6)
- net Top Side/CPIN7: now reaches P?.7 (P7)
- net Top Side/CPIN8: now reaches P?.8 (P8)
- net Top Side/CPIN9: now reaches P?.9 (P9)
Changed lines of the file:
@@
 LIBS:mt48lc32
 LIBS:lm3671mf-fix
+LIBS:h743
 LIBS:helga-cache
 EELAYER 25 0
@@
 encoding utf-8
 Sheet 1 3
-Title ""
-Date ""
-Rev ""
+Title "Helga Palmtop"
+Date "2019-03-27"
+Rev "A"
 Comp ""
 Comment1 ""
@@
 F0 "Top Side" 60
 F1 "top.sch" 60
+F2 "CPIN9" I R 4450 2550 60
+F3 "CPIN10" I R 4450 2650 60
+F4 "CPIN11" I R 4450 2750 60
+F5 "CPIN1" I R 4450 1750 60
+F6 "CPIN2" I R 4450 1850 60
+F7 "CPIN12" I R 4450 2850 60
+F8 "CPIN13" I R 4450 2950 60
+F9 "CPIN14" I R 4450 3050 60
+F10 "CPIN15" I R 4450 3150 60
+F11 "CPIN16" I R 4450 3250 60
+F12 "CPIN3" I R 4450 1950 60
+F13 "CPIN4" I R 4450 2050 60
+F14 "CPIN5" I R 4450 2150 60
+F15 "CPIN6" I R 4450 2250 60
+F16 "CPIN7" I R 4450 2350 60
+F17 "CPIN8" I R 4450 2450 60
+F18 "CPIN17" I R 4450 3350 60
+F19 "CPIN18" I R 4450 3450 60
+F20 "CPIN19" I R 4450 3550 60
+F21 "CPIN20" I R 4450 3650 60
 $EndSheet
 $Sheet
@@
 Wire Wire Line
 	6200 3650 6750 3650
+Wire Wire Line
+	4450 1750 5000 1750
+Wire Wire Line
+	4450 1850 5000 1850
+Wire Wire Line
+	4450 1950 5000 1950
+Wire Wire Line
+	4450 2050 5000 2050
+Wire Wire Line
+	4450 2150 5000 2150
+Wire Wire Line
+	4450 2250 5000 2250
+Wire Wire Line
+	4450 2350 5000 2350
+Wire Wire Line
+	4450 2450 5000 2450
+Wire Wire Line
+	4450 2550 5000 2550
+Wire Wire Line
+	4450 2650 5000 2650
+Wire Wire Line
+	4450 2750 5000 2750
+Wire Wire Line
+	4450 2850 5000 2850
+Wire Wire Line
+	4450 2950 5000 2950
+Wire Wire Line
+	4450 3050 5000 3050
+Wire Wire Line
+	4450 3150 5000 3150
+Wire Wire Line
+	4450 3250 5000 3250
+Wire Wire Line
+	5000 3350 4450 3350
+Wire Wire Line
+	5000 3450 4450 3450
+Wire Wire Line
+	5000 3550 4450 3550
+Wire Wire Line
+	5000 3650 4450 3650
 $EndSCHEMATC
